File: Bridge/Bridge_DS2482.brd (EAGLE design)
At the start: 15 x 20 mm, 20 parts, among them Q1 BSS84, X1 3v3, X10 3v3, X11 3v3, X2 3v3, X3 GND, X4 GND, X5 GND, X6 3v3, X7 GND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

Commit message: Typo correction and more elegance presentation
Parts:
- IC1: value (none) -> DS2482S-100
- R4: value (none) -> /A0
- R5: value (none) -> A0
- R6: value (none) -> A1
- R7: value (none) -> /A1
- X1: value 3v3 -> OW
- X11: value 3v3 -> GND
- X4, X8: value GND -> SCL
- X5, X9: value GND -> SDA
- turned X1 to 180 degrees
- turned X10 to 180 degrees
- turned X11 to 180 degrees
Changed lines of the file:
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@@
 <grid distance="0.127" unitdist="mm" unit="mm" style="lines" multiple="1" display="no" altdistance="0.025" altunitdist="inch" altunit="mm"/>
 <layers>
-<layer number="1" name="Top" color="4" fill="1" visible="yes" active="yes"/>
+<layer number="1" name="Top" color="4" fill="1" visible="no" active="yes"/>
 <layer number="2" name="Route2" color="1" fill="3" visible="no" active="no"/>
 <layer number="3" name="Route3" color="4" fill="3" visible="no" active="no"/>
@@
 <layer number="14" name="Route14" color="1" fill="6" visible="no" active="no"/>
 <layer number="15" name="Route15" color="4" fill="6" visible="no" active="no"/>
-<layer number="16" name="Bottom" color="1" fill="1" visible="yes" active="yes"/>
+<layer number="16" name="Bottom" color="1" fill="1" visible="no" active="yes"/>
 <layer number="17" name="Pads" color="2" fill="1" visible="yes" active="yes"/>
 <layer number="18" name="Vias" color="2" fill="1" visible="yes" active="yes"/>
@@
 <layer number="23" name="tOrigins" color="15" fill="1" visible="yes" active="yes"/>
 <layer number="24" name="bOrigins" color="15" fill="1" visible="no" active="yes"/>
-<layer number="25" name="tNames" color="7" fill="1" visible="no" active="yes"/>
+<layer number="25" name="tNames" color="7" fill="1" visible="yes" active="yes"/>
 <layer number="26" name="bNames" color="7" fill="1" visible="no" active="yes"/>
-<layer number="27" name="tValues" color="7" fill="1" visible="no" active="yes"/>
+<layer number="27" name="tValues" color="7" fill="1" visible="yes" active="yes"/>
 <layer number="28" name="bValues" color="7" fill="1" visible="no" active="yes"/>
 <layer number="29" name="tStop" color="7" fill="3" visible="no" active="yes"/>
@@
 <element name="X2" library="Conn" package="T1.6/0.9" value="3v3" x="3.683" y="2.413" rot="R270"/>
 <element name="X3" library="Conn" package="T1.6/0.9" value="GND" x="6.223" y="2.413" rot="R270"/>
-<element name="X4" library="Conn" package="T1.6/0.9" value="GND" x="8.763" y="2.413" rot="R270"/>
-<element name="X5" library="Conn" package="T1.6/0.9" value="GND" x="11.303" y="2.413" rot="R270"/>
+<element name="X4" library="Conn" package="T1.6/0.9" value="SCL" x="8.763" y="2.413" rot="R270"/>
+<element name="X5" library="Conn" package="T1.6/0.9" value="SDA" x="11.303" y="2.413" rot="R270"/>
 <element name="X6" library="Conn" package="T1.6/0.9" value="3v3" x="3.683" y="17.653" rot="R90"/>
 <element name="X7" library="Conn" package="T1.6/0.9" value="GND" x="6.223" y="17.653" rot="R90"/>
-<element name="X8" library="Conn" package="T1.6/0.9" value="GND" x="8.763" y="17.653" rot="R90"/>
-<element name="X9" library="Conn" package="T1.6/0.9" value="GND" x="11.303" y="17.653" rot="R90"/>
-<element name="IC1" library="maxim" package="SO8" value="" x="8.509" y="9.017" rot="R270"/>
-<element name="R7" library="RCL" package="0603" value="" x="12.954" y="7.112" rot="R270"/>
-<element name="R4" library="RCL" package="0603" value="" x="12.954" y="9.652" rot="R90"/>
-<element name="R5" library="RCL" package="0603" value="" x="11.303" y="11.176" rot="R90"/>
-<element name="R6" library="RCL" package="0603" value="" x="9.906" y="11.176" rot="R90"/>
+<element name="X8" library="Conn" package="T1.6/0.9" value="SCL" x="8.763" y="17.653" rot="R90"/>
+<element name="X9" library="Conn" package="T1.6/0.9" value="SDA" x="11.303" y="17.653" rot="R90"/>
+<element name="IC1" library="maxim" package="SO8" value="DS2482S-100" x="8.509" y="9.017" rot="R270"/>
+<element name="R7" library="RCL" package="0603" value="/A1" x="12.954" y="7.112" rot="R270"/>
+<element name="R4" library="RCL" package="0603" value="/A0" x="12.954" y="9.652" rot="R90"/>
+<element name="R5" library="RCL" package="0603" value="A0" x="11.303" y="11.176" rot="R90"/>
+<element name="R6" library="RCL" package="0603" value="A1" x="9.906" y="11.176" rot="R90"/>
 <element name="Q1" library="Transistor" package="SOT23" value="BSS84" x="7.239" y="11.938" rot="R180"/>
-<element name="X1" library="Conn" package="T1.6/0.9" value="3v3" x="3.683" y="9.017"/>
-<element name="X10" library="Conn" package="T1.6/0.9" value="3v3" x="3.81" y="11.557"/>
-<element name="X11" library="Conn" package="T1.6/0.9" value="3v3" x="3.683" y="6.477"/>
+<element name="X1" library="Conn" package="T1.6/0.9" value="OW" x="3.683" y="9.017" rot="R180"/>
+<element name="X10" library="Conn" package="T1.6/0.9" value="3v3" x="3.81" y="11.557" rot="R180"/>
+<element name="X11" library="Conn" package="T1.6/0.9" value="GND" x="3.683" y="6.477" rot="R180"/>
 </elements>
 <signals>
