File: Bridge/EXT_TWI_LVC.sch (EAGLE design)
At the start: 15 parts, among them IC1 MCP23016-I/SO

Commit message: Added ...
Parts:
- removed R6, R7, R8, R9: cfg, RCL:R0603
- removed SV1: (no value), Conn:ML6ES
- added C3, C4: 1u, RCL:C1206
- added D1: PRLL5819, Diode:D-SCHOTKY7
- added IC2: MC78M05, DCDC:78XXD
- added X1, X13, X5, X9: VCC, Conn:WIREPADT1.6/0.9
- added X10, X14, X2, X6: GND, Conn:WIREPADT1.6/0.9
- added X11, X15, X3, X7: SCL, Conn:WIREPADT1.6/0.9
- added X12, X16, X4, X8: SDA, Conn:WIREPADT1.6/0.9
- C1: value 33p -> 100n
- IC1: value MCP23016-I/SO -> PCA9517; device ICs:MCP23016-I/SO -> Other:PCA9517D
- R1: value 3k9 -> 10k
- R2, R3: value 4k7 -> 10k
- R4: value cfg -> 10k
- R5: value cfg -> n.b.; device RCL:R0603 -> RCL:R1206
Connections:
- removed net +3V3: C2.1, IC1.VDD, IN-11.S, OUT-11.S, R1.2, R2.2, R3.1, R4.1, R5.1, R6.1, SV1-6.S
- removed net N$10: IC1.A0, R4.2, R7.1
- removed net N$11: IC1.A1, R5.2, R8.1
- removed net N$12: IC1.A2, R6.2, R9.1
- removed net N$13: IC1.GP0.0, SV1-1.S
- removed net N$14: IC1.GP0.1, SV1-2.S
- removed net N$15: IC1.GP0.2, SV1-3.S
- removed net N$16: IC1.GP0.3, SV1-4.S
- removed net N$17: IC1.GP0.4, OUT-18.S
- removed net N$18: IC1.GP0.5, OUT-17.S
- removed net N$19: IC1.GP0.6, OUT-16.S
- removed net N$20: IC1.GP0.7, OUT-15.S
- removed net N$4: IC1.GP1.2, OUT-8.S
- removed net N$5: IC1.GP1.1, OUT-9.S
- removed net N$6: IC1.GP1.0, OUT-10.S
- removed net N$7: IC1.GP1.5, OUT-5.S
- removed net N$8: IC1.GP1.6, OUT-4.S
- removed net N$9: IC1.GP1.7, OUT-3.S
- removed net PC4/SDA: IC1.SDA, IN-14.S, OUT-14.S, R3.2
- removed net PC5/SCL: IC1.SCL, IN-13.S, OUT-13.S, R2.1
- removed net VCC: IN-1.S, OUT-1.S
- new net PC0: IN-18.S, OUT-18.S
- new net PC1: IN-17.S, OUT-17.S
- new net PC2: IN-16.S, OUT-16.S
- new net PC3: IN-15.S, OUT-15.S
- new net PD0: IN-10.S, OUT-10.S
- new net PD1: IN-9.S, OUT-9.S
- new net PD2: IN-8.S, OUT-8.S
- new net PD3: IN-7.S, OUT-7.S
- new net PD4: IN-6.S, OUT-6.S
- new net PD5: IN-5.S, OUT-5.S
- new net PD6: IN-4.S, OUT-4.S
- new net PD7: IN-3.S, OUT-3.S
- new net SCLA: IC1.SCLA, IN-13.S, R1.1, X3.S, X7.S
- new net SCLB: IC1.SCLB, OUT-13.S, R3.1, X11.S, X15.S
- new net SDAA: IC1.SDAA, IN-14.S, R2.1, X4.S, X8.S
- new net SDAB: IC1.SDAB, OUT-14.S, R4.1, X12.S, X16.S
- new net VCCA: C1.1, IC1.VCCA, IN-11.S, R1.2, R2.2, R5.2, X1.S, X5.S
- new net VCCB: C2.2, C4.1, IC1.VCCB, IC2.OUT, OUT-11.S, R3.2, R4.2, R5.1, X13.S, X9.S
- new net VIN: D1.A, IN-1.S, OUT-1.S
- net GND: now also C1.2, C2.1, C3.1, C4.2, IC1.GND, IC2.GND, X10.S, X14.S, X2.S, X6.S; no longer C1.1, C2.2, IC1.VSS@1, IC1.VSS@19, IC1.VSS@8, R7.2, R8.2, R9.2, SV1-5.S
- net N$1: now also IN-20.S, OUT-20.S; no longer C1.2, IC1.CLK, R1.1
- net N$2: now also C3.2, D1.C, IC2.IN; no longer IC1.GP1.4, OUT-6.S
- net N$3: now also IN-19.S, OUT-19.S; no longer IC1.GP1.3, OUT-7.S
Other:
- moved on the sheet: C1, C2, IN-1, IN-11, IN-12, IN-13, IN-14, IN-2, OUT-1, OUT-10, OUT-11, OUT-12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
