File: Bridge/EXT_TWI_LVC.brd (EAGLE design)
At the start: 22.5 x 72 mm, 19 parts, among them IC1 TINY45, Q1 IRLU3410, Q2 IRLU3410, Q3 IRLU3410, X2 PW1

Commit message: Added ...
Parts:
- removed LED1: LEDR, Optic:1206
- removed LED2: LEDG, Optic:1206
- removed LED3: LEDB, Optic:1206
- removed Q1, Q2, Q3: IRLU3410, Transistor:TO251AA
- removed R6: 330R, RCL:0603
- removed XS1: 1727049, Conn:1727049
- added C2: 100n, RCL:0603
- added C3, C4: 1u, RCL:1206
- added D1: PRLL5819, Diode:SOD87
- added IC2: MC78M05, DCDC:DPAK
- added X10, X14, X6: GND, Conn:T1.6/0.9
- added X11, X15, X3, X7: SCL, Conn:T1.6/0.9
- added X12, X16, X4, X8: SDA, Conn:T1.6/0.9
- added X13, X5, X9: VCC, Conn:T1.6/0.9
- C1: value 1u -> 100n
- IC1: value TINY45 -> PCA9517; device atmel:SOIC8 -> Other:SOIC8
- R4: value 330R -> 10k
- R5: value 330R -> n.b.; device RCL:0603 -> RCL:1206
- X1: value (none) -> VCC
- X2: value PW1 -> GND
- moved R5 27.8 mm to (13.6, 52.2), turned to 180 degrees
- moved R4 24.2 mm to (20.2, 37.3), turned to 90 degrees
- moved X2 13.6 mm to (10.2, 29.2), turned to 270 degrees
- moved OUT 11.2 mm to (20.7, 56.8)
- moved R2 10.7 mm to (4.95, 37.3), turned to 90 degrees
- moved X1 10.0 mm to (12.7, 29.2), turned to 270 degrees
- moved R1 6.19 mm to (6.35, 37.3), turned to 90 degrees
- moved IC1 5.64 mm to (12.6, 35.9)
- moved C1 3.54 mm to (10.7, 39.5), turned to 0 degrees
- moved R3 3.43 mm to (18.8, 37.3), turned to 90 degrees
Connections:
- removed net +3V3: C1.2, IC1.8, IN.P$11, OUT.P$11, R1.1, R2.1, R3.1
- removed net BLUE: IC1.3, Q3.1, R6.2
- removed net GREEN: IC1.6, Q2.1, R5.2
- removed net N$4: LED1.1, R4.1
- removed net N$5: LED2.1, R5.1
- removed net N$6: Q1.2, XS1.2
- removed net N$7: Q2.2, XS1.3
- removed net N$8: Q3.2, XS1.4
- removed net N$9: LED3.1, R6.1
- removed net PC4/SDA: IC1.5, IN.P$14, OUT.P$14, R3.2
- removed net PC5/SCL: IC1.7, IN.P$13, OUT.P$13, R2.2
- removed net RED: IC1.2, Q1.1, R4.2
- removed net RST: IC1.1, R1.2
- new net N$2: C3.2, D1.C, IC2.1
- new net SCLA: IC1.2, IN.P$13, R1.1, X3.1, X7.1
- new net SCLB: IC1.7, OUT.P$13, R3.1, X11.1, X15.1
- new net SDAA: IC1.3, IN.P$14, R2.1, X4.1, X8.1
- new net SDAB: IC1.6, OUT.P$14, R4.1, X12.1, X16.1
- new net VCCA: C1.1, IC1.1, IN.P$11, R1.2, R2.2, R5.2, X1.1, X5.1
- new net VCCB: C2.2, C4.1, IC1.8, IC2.3, OUT.P$11, R3.2, R4.2, R5.1, X13.1, X9.1
- net GND: now also C1.2, C2.1, C3.1, C4.2, IC2.4, X10.1, X14.1, X2.1, X6.1; no longer C1.1, LED1.2, LED2.2, LED3.2, Q1.3, Q2.3, Q3.3, XS1.1
- net VIN: now also D1.A; no longer X1.1, X2.1, XS1.5
Routing:
- net VIN: track 74.9 -> 17.4 mm
- net VCCB: track 0.00 -> 50.3 mm, vias 0 -> 1
- net VCCA: track 0.00 -> 47.2 mm, vias 0 -> 1
- net SDAB: track 0.00 -> 41.5 mm, vias 0 -> 1
- net SCLB: track 0.00 -> 39.0 mm, vias 0 -> 2
- net SDAA: track 0.00 -> 37.3 mm, vias 0 -> 1
- net SCLA: track 0.00 -> 33.8 mm, vias 0 -> 2
- net +3V3: track 33.1 -> 0.00 mm, vias 1 -> 0
- net PC4/SDA: track 30.8 -> 0.00 mm, vias 1 -> 0
- net RED: track 30.2 -> 0.00 mm, vias 1 -> 0
- net N$8: track 26.1 -> 0.00 mm
- net PC5/SCL: track 22.8 -> 0.00 mm, vias 1 -> 0
- net GREEN: track 21.1 -> 0.00 mm, vias 1 -> 0
- net N$7: track 18.6 -> 0.00 mm
- net BLUE: track 12.7 -> 0.00 mm, vias 1 -> 0
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Other:
- board size 22.5 x 72 mm -> 33.8 x 72 mm
- board text added: "EXT TWI LVC"
- board text added: "GND"
- board text added: "SCL"
- board text added: "SDA"
- board text added: "VCCA"
- board text added: "VCCB"
- board text added: "X13Home.org"
- board text removed: "+"
- board text removed: "0"
- board text removed: "B"
- board text removed: "G"
- board text removed: "R"

Commit message: Reorganization
Parts:
- moved X13 7.62 mm to (20.3, 16.5), turned to 90 degrees
- moved X14 7.62 mm to (22.9, 16.5), turned to 90 degrees
- moved X15 7.62 mm to (25.4, 16.5), turned to 90 degrees
- moved X16 7.62 mm to (27.9, 16.5), turned to 90 degrees
- moved X5 7.62 mm to (12.7, 16.5), turned to 90 degrees
- moved X6 7.62 mm to (10.2, 16.5), turned to 90 degrees
- moved X7 7.62 mm to (7.62, 16.5), turned to 90 degrees
- moved X8 7.62 mm to (5.08, 16.5), turned to 90 degrees
Routing:
- net VCCB: track 50.3 -> 57.9 mm
- net VCCA: track 47.2 -> 54.8 mm
- net SDAA: track 37.3 -> 44.9 mm
- net SCLB: track 39.0 -> 46.6 mm
- net SCLA: track 33.8 -> 41.4 mm
- net SDAB: track 41.5 -> 49.1 mm
