File: Sensors/Sens_BMP085.sch (EAGLE design)
At the start: 15 parts, among them IC1 BMP085, X1 EOC, X12 XCLR, X2 3v3, X3 GND, X4 GND, X5 GND, X6 3v3, X7 GND, X8 GND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

Commit message: Typo correction and more elegance presentation
Parts:
- X4, X8: value GND -> SCL
- X5, X9: value GND -> SDA
Other:
- moved on the sheet: C1, IC1, R1, R2, R3, X1, X12, X2, X3, X4, X5, X6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
