File: Sensors/Sens_BMP085_HIH613x.brd (EAGLE design)
At the start: 20 x 20 mm, 20 parts, among them IC1 BMP085, IC2 HIH613x-021, X1 EOC, X10 ALL, X11 ALH, X12 XCLR, X2 3v3, X3 GND, X4 GND, X5 GND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

Commit message: Typo correction and more elegance presentation
Parts:
- X4, X8: value GND -> SCL
- X5, X9: value GND -> SDA
- turned X4 to 270 degrees
- turned X5 to 270 degrees
- turned X6 to 90 degrees
- turned X7 to 90 degrees
- turned X8 to 90 degrees
- turned X9 to 90 degrees
