File: Sensors/Sens_LM75.brd (EAGLE design)
At the start: 13 x 17 mm, 15 parts, among them IC1 BMP085, X1 EOC, X12 XCLR, X2 3v3, X3 GND, X4 SCL, X5 SDA, X6 3v3, X7 GND, X8 SCL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

Commit message: Typo correction and more elegance presentation
Parts:
- removed X12: XCLR, Conn:S1.27R
- removed X9: SDA, Conn:T1.6/0.9
- added R4: A1, RCL:0603
- added R5: A2, RCL:0603
- added R6: /A2, RCL:0603
- added R7: /A1, RCL:0603
- added R8: /A0, RCL:0603
- IC1: value BMP085 -> LM75; device Sensors:LCC8 -> Sensors:SO8
- R1: value 10k -> A0
- R2, R3: value 10k -> 4k7
- X1: value EOC -> SCL; device Conn:S1.27R -> Conn:T1.6/0.9
- X6: value 3v3 -> SDA
- X7: value GND -> 3v3
- X8: value SCL -> GND
- moved R2 10.9 mm to (2.79, 4.57), turned to 90 degrees
- moved C1 10.3 mm to (10.9, 12.2)
- moved R3 8.92 mm to (4.57, 4.57), turned to 90 degrees
- moved X2 7.75 mm to (10.4, 2.16)
- moved X5 7.49 mm to (2.79, 2.16)
- moved X1 7.24 mm to (5.33, 14.9), turned to 90 degrees
- moved R1 6.02 mm to (5.97, 5.97), turned to 270 degrees
- moved X7 5.21 mm to (10.4, 14.9)
- moved X3 2.67 mm to (7.87, 2.16)
- moved X4 2.41 mm to (5.33, 2.16)
- moved IC1 2.01 mm to (5.84, 10.0), turned to 270 degrees
- moved X8 0.25 mm to (8.00, 14.9)
- moved X6 0.13 mm to (2.79, 14.9)
Connections:
- removed net EOC: IC1.2, X1.1
- removed net XCLR: IC1.8, R1.2, X12.1
- new net N$1: IC1.7, R1.1, R8.2
- new net N$2: IC1.6, R4.1, R7.2
- new net N$3: IC1.5, R5.1, R6.2
- net +3V3: now also IC1.8, R1.2, R4.2, R5.2, X7.1; no longer IC1.3, IC1.4, R1.1, X6.1
- net GND: now also IC1.4, R6.1, R7.1, R8.1, X8.1; no longer IC1.1, X7.1
- net SCL: now also IC1.2, X1.1; no longer IC1.6, X8.1
- net SDA: now also IC1.1, X6.1; no longer IC1.7, X9.1
Routing:
- net N$1: track 0.00 -> 7.30 mm
- net SDA: track 23.3 -> 17.4 mm
- net N$2: track 0.00 -> 5.37 mm
- net XCLR: track 4.44 -> 0.00 mm
- net GND: track 0.00 -> 4.19 mm
- net N$3: track 0.00 -> 3.16 mm
- net SCL: track 23.0 -> 20.5 mm
- net +3V3: track 29.8 -> 27.3 mm
- net EOC: track 1.78 -> 0.00 mm
