File: Sensors/Sens_SI7005.brd (EAGLE design)
At the start: 13 x 17 mm, 13 parts, among them X1 GND, X2 3v3, X3 GND, X4 GND, X5 GND, X6 GND, X7 3v3, X8 GND

Commit message: Typo correction and more elegance presentation
Parts:
- IC2: value (none) -> SI7005
- X1, X4: value GND -> SCL
- X5, X6: value GND -> SDA
- turned X1 to 90 degrees
- turned X4 to 270 degrees
- turned X5 to 270 degrees
- turned X6 to 90 degrees
- turned X7 to 90 degrees
- turned X8 to 90 degrees
Changed lines of the file:
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@@
 <grid distance="0.127" unitdist="mm" unit="mm" style="lines" multiple="1" display="no" altdistance="0.025" altunitdist="inch" altunit="mm"/>
 <layers>
-<layer number="1" name="Top" color="4" fill="1" visible="yes" active="yes"/>
+<layer number="1" name="Top" color="4" fill="1" visible="no" active="yes"/>
 <layer number="2" name="Route2" color="1" fill="3" visible="no" active="no"/>
 <layer number="3" name="Route3" color="4" fill="3" visible="no" active="no"/>
@@
 <layer number="14" name="Route14" color="1" fill="6" visible="no" active="no"/>
 <layer number="15" name="Route15" color="4" fill="6" visible="no" active="no"/>
-<layer number="16" name="Bottom" color="1" fill="1" visible="yes" active="yes"/>
+<layer number="16" name="Bottom" color="1" fill="1" visible="no" active="yes"/>
 <layer number="17" name="Pads" color="2" fill="1" visible="yes" active="yes"/>
 <layer number="18" name="Vias" color="2" fill="1" visible="yes" active="yes"/>
@@
 <layer number="23" name="tOrigins" color="15" fill="1" visible="yes" active="yes"/>
 <layer number="24" name="bOrigins" color="15" fill="1" visible="no" active="yes"/>
-<layer number="25" name="tNames" color="7" fill="1" visible="no" active="yes"/>
+<layer number="25" name="tNames" color="7" fill="1" visible="yes" active="yes"/>
 <layer number="26" name="bNames" color="7" fill="1" visible="no" active="yes"/>
-<layer number="27" name="tValues" color="7" fill="1" visible="no" active="yes"/>
+<layer number="27" name="tValues" color="7" fill="1" visible="yes" active="yes"/>
 <layer number="28" name="bValues" color="7" fill="1" visible="no" active="yes"/>
 <layer number="29" name="tStop" color="7" fill="3" visible="no" active="yes"/>
@@
 <element name="X2" library="Conn" package="T1.6/0.9" value="3v3" x="10.414" y="2.159" rot="R270"/>
 <element name="X3" library="Conn" package="T1.6/0.9" value="GND" x="7.874" y="2.159" rot="R270"/>
-<element name="X4" library="Conn" package="T1.6/0.9" value="GND" x="5.334" y="2.159"/>
-<element name="X5" library="Conn" package="T1.6/0.9" value="GND" x="2.794" y="2.159"/>
-<element name="IC2" library="Sensors" package="QFN24" value="" x="6.731" y="9.271" rot="R270"/>
-<element name="X1" library="Conn" package="T1.6/0.9" value="GND" x="5.334" y="14.859"/>
-<element name="X6" library="Conn" package="T1.6/0.9" value="GND" x="2.794" y="14.859"/>
-<element name="X7" library="Conn" package="T1.6/0.9" value="3v3" x="10.414" y="14.859"/>
-<element name="X8" library="Conn" package="T1.6/0.9" value="GND" x="8.001" y="14.859"/>
+<element name="X4" library="Conn" package="T1.6/0.9" value="SCL" x="5.334" y="2.159" rot="R270"/>
+<element name="X5" library="Conn" package="T1.6/0.9" value="SDA" x="2.794" y="2.159" rot="R270"/>
+<element name="IC2" library="Sensors" package="QFN24" value="SI7005" x="6.731" y="9.271" rot="R270"/>
+<element name="X1" library="Conn" package="T1.6/0.9" value="SCL" x="5.334" y="14.859" rot="R90"/>
+<element name="X6" library="Conn" package="T1.6/0.9" value="SDA" x="2.794" y="14.859" rot="R90"/>
+<element name="X7" library="Conn" package="T1.6/0.9" value="3v3" x="10.414" y="14.859" rot="R90"/>
+<element name="X8" library="Conn" package="T1.6/0.9" value="GND" x="8.001" y="14.859" rot="R90"/>
 </elements>
 <signals>
