File: Mainboards/TRV_RFM23_V0.1.brd (EAGLE design)
At the start: 36 x 28 mm, 21 parts, among them IC2 MEGA328P-AU, IC3 LP2992-IM5-3.3, Q1 IRLML9301, X6 BU-SMA-V

Commit message: Added devices
Parts:
- added R4: n.b, RCL:0603
- RF1: value (none) -> RFM23
Connections:
- net N$10 renamed LED
- net MISO: now also R4.1, R4.2
Routing:
- net MISO: track 13.4 -> 14.3 mm
Changed lines of the file:
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@@
 <layer number="19" name="Unrouted" color="6" fill="1" visible="yes" active="yes"/>
 <layer number="20" name="Dimension" color="15" fill="1" visible="yes" active="yes"/>
-<layer number="21" name="tPlace" color="7" fill="1" visible="no" active="yes"/>
-<layer number="22" name="bPlace" color="7" fill="1" visible="no" active="yes"/>
-<layer number="23" name="tOrigins" color="15" fill="1" visible="no" active="yes"/>
-<layer number="24" name="bOrigins" color="15" fill="1" visible="no" active="yes"/>
+<layer number="21" name="tPlace" color="7" fill="1" visible="yes" active="yes"/>
+<layer number="22" name="bPlace" color="7" fill="1" visible="yes" active="yes"/>
+<layer number="23" name="tOrigins" color="15" fill="1" visible="yes" active="yes"/>
+<layer number="24" name="bOrigins" color="15" fill="1" visible="yes" active="yes"/>
 <layer number="25" name="tNames" color="7" fill="1" visible="no" active="yes"/>
 <layer number="26" name="bNames" color="7" fill="1" visible="no" active="yes"/>
@@
 <element name="QR1" library="QUARTZ" package="CR" value="8M" x="18.034" y="12.827" rot="R180"/>
 <element name="C2" library="RCL" package="SMC_B" value="10u" x="22.606" y="4.699" rot="R270"/>
-<element name="RF1" library="RF" package="RFM23B" value="" x="18.288" y="11.176" rot="MR90"/>
+<element name="RF1" library="RF" package="RFM23B" value="RFM23" x="18.288" y="11.176" rot="MR90"/>
 <element name="X6" library="Conn" package="BU-SMA-V" value="BU-SMA-V" x="31.322" y="14">
 <attribute name="OC_NEWARK" value="unknown" x="31.322" y="14" size="1.778" layer="27" display="off"/>
@@
 <attribute name="OC_FARNELL" value="unknown" x="31.322" y="14" size="1.778" layer="27" display="off"/>
 </element>
+<element name="R4" library="RCL" package="0603" value="n.b" x="13.97" y="21.209" rot="MR0"/>
 </elements>
 <signals>
@@
 <wire x1="24.13" y1="24.765" x2="24.13" y2="25.4" width="0.4064" layer="1"/>
 <contactref element="RF1" pad="11"/>
-<wire x1="15.288" y1="19.076" x2="15.288" y2="19.733" width="0.4064" layer="16"/>
-<wire x1="15.288" y1="19.733" x2="17.018" y2="21.463" width="0.4064" layer="16"/>
-<wire x1="17.018" y1="21.463" x2="22.098" y2="21.463" width="0.4064" layer="16"/>
+<wire x1="16.764" y1="21.463" x2="22.098" y2="21.463" width="0.4064" layer="16"/>
 <wire x1="22.098" y1="21.463" x2="22.86" y2="22.225" width="0.4064" layer="16"/>
 <wire x1="22.86" y1="22.225" x2="22.86" y2="23.622" width="0.254" layer="16"/>
 <wire x1="22.86" y1="23.622" x2="24.13" y2="24.892" width="0.4064" layer="16"/>
 <wire x1="24.13" y1="24.892" x2="24.13" y2="25.4" width="0.4064" layer="16"/>
+<wire x1="15.288" y1="19.076" x2="15.288" y2="19.352" width="0.4064" layer="16"/>
+<wire x1="15.288" y1="19.352" x2="15.748" y2="19.812" width="0.4064" layer="16"/>
+<wire x1="15.748" y1="19.812" x2="15.748" y2="20.447" width="0.4064" layer="16"/>
+<wire x1="15.748" y1="20.447" x2="16.764" y2="21.463" width="0.4064" layer="16"/>
 </signal>
 <signal name="SCK">
@@
 <wire x1="20.4216" y1="23.5966" x2="20.955" y2="24.13" width="0.4064" layer="1"/>
 <contactref element="RF1" pad="12"/>
-<wire x1="17.288" y1="19.076" x2="17.288" y2="19.701" width="0.4064" layer="16"/>
-<wire x1="17.288" y1="19.701" x2="18.288" y2="20.701" width="0.4064" layer="16"/>
-<wire x1="18.288" y1="20.701" x2="22.352" y2="20.701" width="0.4064" layer="16"/>
+<wire x1="18.034" y1="20.701" x2="22.352" y2="20.701" width="0.4064" layer="16"/>
 <wire x1="22.352" y1="20.701" x2="24.13" y2="22.479" width="0.4064" layer="16"/>
 <wire x1="24.13" y1="22.479" x2="24.13" y2="22.86" width="0.4064" layer="16"/>
+<wire x1="17.288" y1="19.076" x2="17.288" y2="19.32" width="0.4064" layer="16"/>
+<wire x1="17.288" y1="19.32" x2="17.78" y2="19.812" width="0.4064" layer="16"/>
+<wire x1="17.78" y1="19.812" x2="17.78" y2="20.447" width="0.4064" layer="16"/>
+<wire x1="17.78" y1="20.447" x2="18.034" y2="20.701" width="0.4064" layer="16"/>
 </signal>
 <signal name="RSEL">
@@
 <wire x1="20.834" y1="22.104" x2="21.59" y2="22.86" width="0.4064" layer="1"/>
 <contactref element="RF1" pad="10"/>
-<wire x1="13.288" y1="19.076" x2="13.288" y2="19.765" width="0.4064" layer="16"/>
-<wire x1="13.288" y1="19.765" x2="15.748" y2="22.225" width="0.4064" layer="16"/>
-<wire x1="15.748" y1="22.225" x2="20.955" y2="22.225" width="0.4064" layer="16"/>
+<contactref element="R4" pad="1"/>
+<contactref element="R4" pad="2"/>
+<wire x1="13.288" y1="19.076" x2="13.288" y2="21.1936" width="0.4064" layer="16"/>
+<wire x1="13.288" y1="21.1936" x2="13.2726" y2="21.209" width="0.4064" layer="16"/>
+<wire x1="13.2726" y1="21.209" x2="14.6674" y2="21.209" width="0.4064" layer="16"/>
+<wire x1="14.6674" y1="21.209" x2="15.494" y2="21.209" width="0.4064" layer="16"/>
+<wire x1="15.494" y1="21.209" x2="16.51" y2="22.225" width="0.4064" layer="16"/>
+<wire x1="16.51" y1="22.225" x2="20.955" y2="22.225" width="0.4064" layer="16"/>
 <wire x1="20.955" y1="22.225" x2="21.59" y2="22.86" width="0.4064" layer="16"/>
 </signal>
@@
 <wire x1="5.08" y1="2.54" x2="7.3036" y2="2.54" width="0.6096" layer="1"/>
 </signal>
-<signal name="N$10">
+<signal name="LED">
 <contactref element="IC2" pad="12"/>
 <contactref element="R5" pad="1"/>
