File: Mainboards/S2EC13.brd (EAGLE design)
At the start: 43 x 72 mm, 47 parts, among them CN2 SWD, IC1 LD1117S33, IC2 CC1101RTK, IC3 STM32F051C8, Q1 IRLML9301, Q2 8M, X3 SMA-BU

Commit message: S2EC13, corrected R9
Parts:
- R9: value 0R -> NC
Changed lines of the file:
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@@
 <element name="C15" library="RCL" package="0603" value="10n" x="24.765" y="56.769" rot="R180"/>
 <element name="R7" library="RCL" package="0603" value="0R" x="17.399" y="64.516" rot="MR270"/>
-<element name="R9" library="RCL" package="0603" value="0R" x="16.637" y="68.199" rot="R180"/>
+<element name="R9" library="RCL" package="0603" value="NC" x="16.637" y="68.199" rot="R180"/>
 </elements>
 <signals>
