File: Mainboards/S2EC13.sch (EAGLE design)
At the start: 47 parts, among them CN2 SWD, IC1 LD1117S33, IC2 CC1101RTK, IC3 STM32F051C8, Q1 IRLML9301, Q2 8M, X3 SMA-BU

Commit message: S2EC13, corrected R9
Parts:
- R9: value 0R -> NC
Changed lines of the file:
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@@
 <part name="+3V10" library="supply1" deviceset="+3V3" device=""/>
 <part name="R7" library="RCL" deviceset="R" device="0603" value="0R"/>
-<part name="R9" library="RCL" deviceset="R" device="0603" value="0R"/>
+<part name="R9" library="RCL" deviceset="R" device="0603" value="NC"/>
 </parts>
 <sheets>
