File: Mainboards/S2Mn10.brd (EAGLE design)
At the start: 33 x 19 mm, 34 parts, among them IC1 STM32F051K8, IC2 SN65HVD72DR, IC4 TPS70933, Q1 8M, X1 P0, X10 SDA, X11 SWD, X12 GND, X13 SWC, X14 3V3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

Commit message: Minor Changes
Changed lines of the file:
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@@
 <grid distance="0.127" unitdist="mm" unit="mm" style="lines" multiple="1" display="no" altdistance="0.025" altunitdist="inch" altunit="inch"/>
 <layers>
-<layer number="1" name="Top" color="4" fill="1" visible="no" active="yes"/>
+<layer number="1" name="Top" color="4" fill="1" visible="yes" active="yes"/>
 <layer number="2" name="Route2" color="1" fill="3" visible="no" active="no"/>
 <layer number="3" name="Route3" color="4" fill="3" visible="no" active="no"/>
@@
 <layer number="22" name="bPlace" color="7" fill="1" visible="no" active="yes"/>
 <layer number="23" name="tOrigins" color="15" fill="1" visible="no" active="yes"/>
-<layer number="24" name="bOrigins" color="15" fill="1" visible="yes" active="yes"/>
+<layer number="24" name="bOrigins" color="15" fill="1" visible="no" active="yes"/>
 <layer number="25" name="tNames" color="7" fill="1" visible="no" active="yes"/>
-<layer number="26" name="bNames" color="7" fill="1" visible="yes" active="yes"/>
+<layer number="26" name="bNames" color="7" fill="1" visible="no" active="yes"/>
 <layer number="27" name="tValues" color="7" fill="1" visible="no" active="yes"/>
-<layer number="28" name="bValues" color="7" fill="1" visible="yes" active="yes"/>
+<layer number="28" name="bValues" color="7" fill="1" visible="no" active="yes"/>
 <layer number="29" name="tStop" color="7" fill="3" visible="no" active="yes"/>
 <layer number="30" name="bStop" color="7" fill="6" visible="no" active="yes"/>
@@
 <wire x1="27.432" y1="4.375" x2="29.775" y2="4.375" width="0.6096" layer="1"/>
 <wire x1="29.775" y1="4.375" x2="29.845" y2="4.445" width="0.6096" layer="1"/>
-<wire x1="31.75" y1="5.842" x2="30.353" y2="4.445" width="0.4064" layer="1"/>
+<wire x1="31.496" y1="11.373" x2="31.496" y2="5.588" width="0.4064" layer="1"/>
+<wire x1="31.496" y1="5.588" x2="30.353" y2="4.445" width="0.4064" layer="1"/>
 <wire x1="30.353" y1="4.445" x2="29.845" y2="4.445" width="0.4064" layer="1"/>
-<wire x1="31.496" y1="11.373" x2="31.75" y2="11.119" width="0.4064" layer="1"/>
-<wire x1="31.75" y1="11.119" x2="31.75" y2="5.842" width="0.4064" layer="1"/>
 </signal>
 <signal name="LED">

Commit message: Updated mainboards
Parts:
- removed X12: GND, Conn:T1.6/0.9
- removed X14, X17: 3V3, Conn:T1.6/0.9
- added X114, X22: GND, Conn:T1.6/0.9
- added X21: SWC, Conn:T1.6/0.9
- X10: value SDA -> 3V3
- X13: value SWC -> 3V3
- X16: value GND -> SDA
- moved X10 19.8 mm to (24.8, 1.91), turned to 90 degrees
- moved X9 12.4 mm to (22.2, 1.91), turned to 90 degrees
- moved X16 5.08 mm to (12.1, 17.1)
- moved X13 3.05 mm to (19.7, 17.1), turned to 180 degrees
- renumbered X11 to X23
Connections:
- net +3V3: now also X10.1, X13.1; no longer X14.1, X17.1
- net GND: now also X114.1, X22.1; no longer X12.1, X16.1
- net SDA1: now also X16.1; no longer X10.1
- net SWC: now also X21.1; no longer X13.1
