File: Mainboards/S4CX11.brd (EAGLE design)
At the start: 30 x 28 mm, 35 parts, among them IC1 STM32F303K8, Q1 8M

Commit message: Updated mainboards
Connections:
- net DE: now also IC1.22; no longer IC1.21
Changed lines of the file:
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@@
 </signal>
 <signal name="DE">
-<contactref element="IC1" pad="21"/>
 <contactref element="DE" pad="1"/>
-<wire x1="19.921" y1="16.275" x2="22.841" y2="16.275" width="0.4064" layer="1"/>
-<wire x1="22.841" y1="16.275" x2="27.686" y2="11.43" width="0.4064" layer="1"/>
+<wire x1="22.041" y1="17.075" x2="27.686" y2="11.43" width="0.4064" layer="1"/>
 <wire x1="27.686" y1="11.43" x2="27.686" y2="10.795" width="0.4064" layer="1"/>
+<contactref element="IC1" pad="22"/>
+<wire x1="19.921" y1="17.075" x2="22.041" y2="17.075" width="0.4064" layer="1"/>
 </signal>
 <signal name="RX1">
