File: Mainboards/S4QX11.brd (EAGLE design)
At the start: 30 x 28 mm, 37 parts, among them IC1 STM32F303K8, Q1 8M

Commit message: Updated mainboards
Connections:
- net DE: now also IC1.22; no longer IC1.21
Changed lines of the file:
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@@
 <setting verticaltext="up"/>
 </settings>
-<grid distance="5" unitdist="mil" unit="mil" style="lines" multiple="1" display="no" altdistance="0.025" altunitdist="inch" altunit="inch"/>
+<grid distance="5" unitdist="mil" unit="mm" style="lines" multiple="1" display="no" altdistance="0.025" altunitdist="inch" altunit="inch"/>
 <layers>
 <layer number="1" name="Top" color="4" fill="1" visible="yes" active="yes"/>
@@
 <layer number="14" name="Route14" color="1" fill="6" visible="no" active="no"/>
 <layer number="15" name="Route15" color="4" fill="6" visible="no" active="no"/>
-<layer number="16" name="Bottom" color="1" fill="1" visible="yes" active="yes"/>
+<layer number="16" name="Bottom" color="1" fill="1" visible="no" active="yes"/>
 <layer number="17" name="Pads" color="2" fill="1" visible="yes" active="yes"/>
 <layer number="18" name="Vias" color="2" fill="1" visible="yes" active="yes"/>
@@
 <wire x1="20.32" y1="15.24" x2="20.447" y2="15.367" width="0.4064" layer="1"/>
 <wire x1="20.447" y1="15.367" x2="20.828" y2="15.748" width="0.3048" layer="1"/>
-<wire x1="20.828" y1="15.748" x2="23.495" y2="18.415" width="0.4064" layer="1"/>
-<wire x1="23.495" y1="18.415" x2="27.686" y2="18.415" width="0.4064" layer="1"/>
+<wire x1="20.828" y1="15.748" x2="20.955" y2="15.875" width="0.4064" layer="1"/>
+<wire x1="20.955" y1="15.875" x2="25.146" y2="15.875" width="0.4064" layer="1"/>
+<wire x1="25.146" y1="15.875" x2="27.686" y2="18.415" width="0.4064" layer="1"/>
 </signal>
 <signal name="N$1">
@@
 </signal>
 <signal name="DE">
-<contactref element="IC1" pad="21"/>
 <contactref element="DE" pad="1"/>
-<wire x1="21.572" y1="12.592" x2="25.889" y2="12.592" width="0.4064" layer="1"/>
-<wire x1="25.889" y1="12.592" x2="27.686" y2="10.795" width="0.4064" layer="1"/>
+<wire x1="25.089" y1="13.392" x2="27.686" y2="10.795" width="0.4064" layer="1"/>
+<contactref element="IC1" pad="22"/>
+<wire x1="21.572" y1="13.392" x2="25.089" y2="13.392" width="0.4064" layer="1"/>
 </signal>
 <signal name="RX1">
