File: Other/EXT_EXPANDER.brd (EAGLE design)
At the start: 22.5 x 72 mm, 15 parts, among them IC1 MCP23016-I/SO

Commit message: Added ...
Parts:
- removed XS2: 1727049, Conn:1727049
- added SV1: (no value), Conn:ML6S
- IN: device Conn:FE10-2WS -> Conn:FE10-2WSS
Connections:
- net +3V3: now also SV1.6
- net GND: now also SV1.5; no longer XS2.1
- net N$13: now also SV1.1; no longer XS2.2
- net N$14: now also SV1.2; no longer XS2.3
- net N$15: now also SV1.3; no longer XS2.4
- net N$16: now also SV1.4; no longer XS2.5
Routing:
- net +3V3: track 44.8 -> 67.7 mm, vias 0 -> 1
- net N$16: track 30.3 -> 17.7 mm
- net N$15: track 26.5 -> 22.5 mm
- net N$13: track 28.3 -> 25.2 mm
- net N$14: track 22.4 -> 20.7 mm
- net N$23: track 0.00 -> 1.27 mm
- net N$22: track 0.00 -> 1.27 mm
- net N$21: track 0.00 -> 1.27 mm
Other:
- board text added: "BUS Expander"
- board text added: "X13Home.org"
- board text removed: "BUS Extender"
