File: Other/EXT_SCR.brd (EAGLE design)
At the start: 45 x 72 mm, 31 parts, among them Q1 BC817, Q2 BC817, Q3 BC817, Q4 BC817

Commit message: Reorganization
Parts:
- IN: device Conn:FE10-2WS -> Conn:FE10-2WSS
Routing:
- net VCC: track 108.2 -> 104.5 mm
Other:
- board text added: "X13Home.org"
Changed lines of the file:
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@@
 <text x="38.1" y="69.014" size="2.54" layer="1" font="vector" ratio="15">TOP</text>
 <text x="44.577" y="69.035" size="2.54" layer="16" font="vector" ratio="15" rot="MR0">BOT</text>
-<text x="25.4" y="64.008" size="1.778" layer="16" font="vector" ratio="15" rot="MR0">EXT SCR</text>
+<text x="25.4" y="64.008" size="1.778" layer="26" font="vector" ratio="15" rot="MR0">EXT SCR</text>
+<text x="33.274" y="25.654" size="2.54" layer="26" rot="MR0">X13Home.org</text>
 </plain>
 <attributes>
@@
 <elements>
 <element name="OUT" library="Conn" package="ML20LS" value="MF20" x="31.877" y="56.769" rot="R270"/>
-<element name="IN" library="Conn" package="FE10-2WS" value="EF20" x="3.81" y="56.769" rot="R270"/>
+<element name="IN" library="Conn" package="FE10-2WSS" value="EF20" x="3.81" y="56.769" rot="R270"/>
 <element name="SCR1" library="Relay_Switch" package="S202" value="S202S02" x="6.35" y="26.67" rot="R90"/>
-<element name="R1" library="RCL" package="0603" value="47R" x="4.699" y="36.83"/>
+<element name="R1" library="RCL" package="0603" value="47R" x="4.699" y="36.83" smashed="yes">
+<attribute name="VALUE" x="3.974" y="36.627" size="0.254" layer="27" ratio="10"/>
+<attribute name="NAME" x="2.032" y="36.449" size="0.8128" layer="25" ratio="10"/>
+</element>
 <element name="R2" library="RCL" package="0603" value="180R" x="4.699" y="38.227"/>
 <element name="LED1" library="Optic" package="1206" value="LEDR" x="2.286" y="39.751" rot="R90"/>
-<element name="Q1" library="Transistor" package="SOT23" value="BC817" x="8.128" y="37.846" rot="R270"/>
-<element name="R3" library="RCL" package="0603" value="10k" x="8.89" y="40.259" rot="R180"/>
-<element name="R4" library="RCL" package="0603" value="1k" x="6.858" y="40.894" rot="R270"/>
+<element name="Q1" library="Transistor" package="SOT23" value="BC817" x="8.128" y="37.846" smashed="yes" rot="R270">
+<attribute name="NAME" x="10.16" y="36.195" size="0.8128" layer="25"/>
+<attribute name="VALUE" x="8.007" y="39.078" size="0.254" layer="27" rot="R270"/>
+</element>
+<element name="R3" library="RCL" package="0603" value="10k" x="8.89" y="40.259" smashed="yes" rot="R180">
+<attribute name="VALUE" x="9.615" y="40.462" size="0.254" layer="27" ratio="10" rot="R180"/>
+<attribute name="NAME" x="10.16" y="41.783" size="0.8128" layer="25" ratio="10" rot="R180"/>
+</element>
+<element name="R4" library="RCL" package="0603" value="1k" x="6.858" y="40.894" smashed="yes" rot="R270">
+<attribute name="VALUE" x="6.655" y="41.619" size="0.254" layer="27" ratio="10" rot="R270"/>
+<attribute name="NAME" x="5.334" y="42.164" size="0.8128" layer="25" ratio="10" rot="R270"/>
+</element>
 <element name="SCR2" library="Relay_Switch" package="S202" value="S202S02" x="16.51" y="26.67" rot="R90"/>
-<element name="R5" library="RCL" package="0603" value="47R" x="14.986" y="36.83"/>
+<element name="R5" library="RCL" package="0603" value="47R" x="14.986" y="36.83" smashed="yes">
+<attribute name="VALUE" x="14.261" y="36.627" size="0.254" layer="27" ratio="10"/>
+<attribute name="NAME" x="12.192" y="36.449" size="0.8128" layer="25" ratio="10"/>
+</element>
 <element name="R6" library="RCL" package="0603" value="180R" x="14.986" y="38.227"/>
 <element name="LED2" library="Optic" package="1206" value="LEDR" x="12.573" y="39.751" rot="R90"/>
-<element name="Q2" library="Transistor" package="SOT23" value="BC817" x="18.288" y="37.846" rot="R270"/>
-<element name="R7" library="RCL" package="0603" value="10k" x="19.05" y="40.259" rot="R180"/>
-<element name="R8" library="RCL" package="0603" value="1k" x="17.018" y="40.894" rot="R270"/>
+<element name="Q2" library="Transistor" package="SOT23" value="BC817" x="18.288" y="37.846" smashed="yes" rot="R270">
+<attribute name="NAME" x="20.32" y="36.195" size="0.8128" layer="25"/>
+<attribute name="VALUE" x="18.167" y="39.078" size="0.254" layer="27" rot="R270"/>
+</element>
+<element name="R7" library="RCL" package="0603" value="10k" x="19.05" y="40.259" smashed="yes" rot="R180">
+<attribute name="VALUE" x="19.775" y="40.462" size="0.254" layer="27" ratio="10" rot="R180"/>
+<attribute name="NAME" x="20.447" y="41.783" size="0.8128" layer="25" ratio="10" rot="R180"/>
+</element>
+<element name="R8" library="RCL" package="0603" value="1k" x="17.018" y="40.894" smashed="yes" rot="R270">
+<attribute name="VALUE" x="16.815" y="41.619" size="0.254" layer="27" ratio="10" rot="R270"/>
+<attribute name="NAME" x="17.78" y="42.418" size="0.8128" layer="25" ratio="10" rot="R270"/>
+</element>
 <element name="SCR3" library="Relay_Switch" package="S202" value="S202S02" x="26.67" y="26.67" rot="R90"/>
-<element name="R9" library="RCL" package="0603" value="47R" x="25.146" y="36.83"/>
+<element name="R9" library="RCL" package="0603" value="47R" x="25.146" y="36.83" smashed="yes">
+<attribute name="VALUE" x="24.421" y="36.627" size="0.254" layer="27" ratio="10"/>
+<attribute name="NAME" x="22.352" y="36.449" size="0.8128" layer="25" ratio="10"/>
+</element>
 <element name="R10" library="RCL" package="0603" value="180R" x="25.146" y="38.227"/>
 <element name="LED3" library="Optic" package="1206" value="LEDR" x="22.733" y="39.751" rot="R90"/>
-<element name="Q3" library="Transistor" package="SOT23" value="BC817" x="28.448" y="37.846" rot="R270"/>
-<element name="R11" library="RCL" package="0603" value="10k" x="29.21" y="40.259" rot="R180"/>
-<element name="R12" library="RCL" package="0603" value="1k" x="27.178" y="40.894" rot="R270"/>
+<element name="Q3" library="Transistor" package="SOT23" value="BC817" x="28.448" y="37.846" smashed="yes" rot="R270">
+<attribute name="NAME" x="30.48" y="36.195" size="0.8128" layer="25"/>
+<attribute name="VALUE" x="28.327" y="39.078" size="0.254" layer="27" rot="R270"/>
+</element>
+<element name="R11" library="RCL" package="0603" value="10k" x="29.21" y="40.259" smashed="yes" rot="R180">
+<attribute name="VALUE" x="29.935" y="40.462" size="0.254" layer="27" ratio="10" rot="R180"/>
+<attribute name="NAME" x="30.988" y="41.783" size="0.8128" layer="25" ratio="10" rot="R180"/>
+</element>
+<element name="R12" library="RCL" package="0603" value="1k" x="27.178" y="40.894" smashed="yes" rot="R270">
+<attribute name="VALUE" x="26.975" y="41.619" size="0.254" layer="27" ratio="10" rot="R270"/>
+<attribute name="NAME" x="27.94" y="43.053" size="0.8128" layer="25" ratio="10" rot="R270"/>
+</element>
 <element name="SCR4" library="Relay_Switch" package="S202" value="S202S02" x="36.83" y="26.67" rot="R90"/>
-<element name="R13" library="RCL" package="0603" value="47R" x="35.433" y="36.83"/>
+<element name="R13" library="RCL" package="0603" value="47R" x="35.433" y="36.83" smashed="yes">
+<attribute name="VALUE" x="34.708" y="36.627" size="0.254" layer="27" ratio="10"/>
+<attribute name="NAME" x="32.131" y="36.449" size="0.8128" layer="25" ratio="10"/>
+</element>
 <element name="R14" library="RCL" package="0603" value="180R" x="35.433" y="38.227"/>
 <element name="LED4" library="Optic" package="1206" value="LEDR" x="33.02" y="39.751" rot="R90"/>
-<element name="Q4" library="Transistor" package="SOT23" value="BC817" x="38.735" y="37.846" rot="R270"/>
-<element name="R15" library="RCL" package="0603" value="10k" x="39.497" y="40.259" rot="R180"/>
-<element name="R16" library="RCL" package="0603" value="1k" x="37.465" y="40.894" rot="R270"/>
+<element name="Q4" library="Transistor" package="SOT23" value="BC817" x="38.735" y="37.846" smashed="yes" rot="R270">
+<attribute name="NAME" x="40.767" y="36.195" size="0.8128" layer="25"/>
+<attribute name="VALUE" x="38.614" y="39.078" size="0.254" layer="27" rot="R270"/>
+</element>
+<element name="R15" library="RCL" package="0603" value="10k" x="39.497" y="40.259" smashed="yes" rot="R180">
+<attribute name="VALUE" x="40.222" y="40.462" size="0.254" layer="27" ratio="10" rot="R180"/>
+<attribute name="NAME" x="41.275" y="41.783" size="0.8128" layer="25" ratio="10" rot="R180"/>
+</element>
+<element name="R16" library="RCL" package="0603" value="1k" x="37.465" y="40.894" smashed="yes" rot="R270">
+<attribute name="VALUE" x="37.262" y="41.619" size="0.254" layer="27" ratio="10" rot="R270"/>
+<attribute name="NAME" x="38.227" y="43.053" size="0.8128" layer="25" ratio="10" rot="R270"/>
+</element>
 <element name="XS1" library="Conn" package="W237-8P" value="1729186" x="22.479" y="11.049"/>
 </elements>
@@
 <wire x1="9.398" y1="36.322" x2="19.558" y2="36.322" width="0.6096" layer="16"/>
 <wire x1="19.558" y1="36.322" x2="29.591" y2="36.322" width="0.6096" layer="16"/>
-<wire x1="29.591" y1="36.322" x2="39.878" y2="36.322" width="0.6096" layer="16"/>
-<wire x1="39.878" y1="36.322" x2="41.021" y2="36.322" width="0.6096" layer="16"/>
-<wire x1="41.021" y1="36.322" x2="42.545" y2="37.846" width="0.6096" layer="16"/>
-<wire x1="42.545" y1="37.846" x2="42.545" y2="63.881" width="0.6096" layer="16"/>
-<wire x1="42.545" y1="63.881" x2="35.941" y2="70.485" width="0.6096" layer="16"/>
-<wire x1="35.941" y1="70.485" x2="31.623" y2="70.485" width="0.6096" layer="16"/>
+<wire x1="29.591" y1="36.322" x2="38.989" y2="36.322" width="0.6096" layer="16"/>
+<wire x1="35.179" y1="70.485" x2="31.623" y2="70.485" width="0.6096" layer="16"/>
 <wire x1="31.623" y1="70.485" x2="30.607" y2="69.469" width="0.6096" layer="16"/>
 <wire x1="30.607" y1="69.469" x2="30.607" y2="68.199" width="0.6096" layer="16"/>
@@
 <wire x1="39.878" y1="37.846" x2="39.878" y2="36.322" width="0.6096" layer="1"/>
 <via x="39.878" y="36.322" extent="1-16" drill="0.6" diameter="1.27"/>
+<wire x1="39.878" y1="36.322" x2="38.989" y2="36.322" width="0.6096" layer="16"/>
+<wire x1="38.989" y1="36.322" x2="38.989" y2="66.675" width="0.6096" layer="16"/>
+<wire x1="38.989" y1="66.675" x2="35.179" y2="70.485" width="0.6096" layer="16"/>
 </signal>
 <signal name="N$1">
