File: Other/EXT_ADIN.brd (EAGLE design)
At the start: 33.8 x 72 mm, 59 parts, among them Q1 BSS139, Q2 BSS139, Q3 BSS139, Q4 BSS139, Q5 BSS139, Q6 BSS139

Commit message: Reorganization
Parts:
- moved C2 0.13 mm to (9.02, 25.7)
- renumbered ZD1 to D1, ZD2 to D2, ZD3 to D3, ZD4 to D4, ZD5 to D5, ZD6 to D6
Other:
- board text added: "X13Home.org"

Commit message: Optimized R
Parts:
- D1, D2, D3, D4, D5, D6: value (none) -> ZMM3,3
- R1.1, R1.2: value 3k3 -> 1k5
- R1.3, R1.4, R1.5, R1.6: value 39k -> n.b.
- R2.1, R2.2: value 6k8 -> 12k
- R2.3, R2.4, R2.5, R2.6: value 10k -> 1k
- R3.2: value 560R -> 510R
- R3.3, R3.4: value 3k6 -> n.b.
- R4.5, R4.6: value 3k6 -> 3k3

Commit message: Added AC Dimmer
Parts:
- R1.3, R1.4: value n.b. -> 2k2
Changed lines of the file:
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@@
 <attribute name="NAME" x="8.406" y="6.604" size="0.8128" layer="25" ratio="10" rot="R270"/>
 </element>
-<element name="R1.3" library="RCL" package="1206" value="n.b." x="14.097" y="23.241" smashed="yes" rot="R180">
+<element name="R1.3" library="RCL" package="1206" value="2k2" x="14.097" y="23.241" smashed="yes" rot="R180">
 <attribute name="VALUE" x="14.986" y="23.351" size="0.3048" layer="27" ratio="10" rot="R180"/>
 <attribute name="NAME" x="15.24" y="23.725" size="0.8128" layer="25" ratio="10" rot="R180"/>
@@
 <attribute name="NAME" x="16.026" y="6.604" size="0.8128" layer="25" ratio="10" rot="R270"/>
 </element>
-<element name="R1.4" library="RCL" package="1206" value="n.b." x="19.177" y="23.241" smashed="yes" rot="R180">
+<element name="R1.4" library="RCL" package="1206" value="2k2" x="19.177" y="23.241" smashed="yes" rot="R180">
 <attribute name="VALUE" x="20.066" y="23.351" size="0.3048" layer="27" ratio="10" rot="R180"/>
 <attribute name="NAME" x="20.32" y="23.725" size="0.8128" layer="25" ratio="10" rot="R180"/>
