File: Other/EXT_LED_RGB_NPN.brd (EAGLE design)
At the start: 22.5 x 72 mm, 19 parts, among them IC1 TINY45, Q1 IRLU3410, Q2 IRLU3410, Q3 IRLU3410, X2 PW1

Commit message: USB Adepter V1
Parts:
- IC1: value TINY45 -> TINY45S
Connections:
- net BLUE: now also IC1.6; no longer IC1.3
- net GREEN: now also IC1.3; no longer IC1.6
Routing:
- net BLUE: track 12.7 -> 9.90 mm
- net GREEN: track 21.1 -> 19.8 mm
