File: Other/EXT_LED_RGB_NPN.sch (EAGLE design)
At the start: 19 parts, among them IC1 TINY45, Q1 IRLU3410, Q2 IRLU3410, Q3 IRLU3410, X2 PW1

Commit message: USB Adepter V1
Parts:
- IC1: value TINY45 -> TINY45S; device atmel:TINY15LS -> atmel:TINY45S
Connections:
- net BLUE: now also IC1.PB1; no longer IC1.(ADC2)PB3
- net GREEN: now also IC1.PB4; no longer IC1.(OCP)PB1
- net PC4/SDA: now also IC1.PB0; no longer IC1.(AREF)PB0
- net PC5/SCL: now also IC1.PB2; no longer IC1.(ADC1)PB2
- net RED: now also IC1.PB3; no longer IC1.(ADC3)PB4
- net RST: now also IC1.PB5; no longer IC1.(ADC0)PB5
