File: Other/EXT_LED.brd (EAGLE design)
At the start: 72 x 33.8 mm, 39 parts

Commit message: Minor Changes
Parts:
- removed LED1, LED2: (no value), Optic:0603
- removed R10, R11: 330R, RCL:0603
- removed SV1: (no value), Conn:ML6S
Connections:
- removed net N$13: LED1.1, SV1.1
- removed net N$14: LED1.2, R10.2
- removed net N$15: LED2.2, R11.2
- removed net N$29: LED2.1, SV1.2
- removed net N$30: LED3.1, SV1.3
- removed net N$31: LED4.1, SV1.4
- net GND: no longer R10.1, R11.1, SV1.5
- net N$1: now also LED4.1
- net N$2: now also LED3.1
Routing:
- net N$31: track 28.0 -> 0.00 mm
- net N$30: track 19.3 -> 0.00 mm
- net N$13: track 10.3 -> 0.00 mm
- net N$2: track 20.7 -> 30.4 mm
- net N$29: track 9.08 -> 0.00 mm
- net N$1: track 14.4 -> 20.8 mm
- net N$15: track 1.15 -> 0.00 mm
- net N$14: track 1.15 -> 0.00 mm
Changed lines of the file:
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@@
 <?xml version="1.0" encoding="utf-8"?>
 <!DOCTYPE eagle SYSTEM "eagle.dtd">
-<eagle version="7.4.0">
+<eagle version="7.5.0">
 <drawing>
 <settings>
@@
 </element>
 <element name="IN" library="Conn" package="FE10-2WSS" value="EF20" x="15.24" y="3.81"/>
-<element name="SV1" library="Conn" package="ML6S" value="" x="37.964" y="11.176" smashed="yes" rot="R90">
-<attribute name="NAME" x="40.25" y="6.858" size="0.8128" layer="25" ratio="10" rot="R180"/>
-<attribute name="VALUE" x="40.25" y="10.033" size="0.4064" layer="27" ratio="10" rot="R90"/>
-</element>
-<element name="LED1" library="Optic" package="0603" value="" x="30.48" y="12.192" rot="R90"/>
-<element name="R10" library="RCL" package="0603" value="330R" x="30.48" y="14.732" rot="R270"/>
-<element name="LED2" library="Optic" package="0603" value="" x="29.21" y="12.192" rot="R90"/>
-<element name="R11" library="RCL" package="0603" value="330R" x="29.21" y="14.732" rot="R270"/>
 <element name="LED3" library="Optic" package="0603" value="" x="27.94" y="12.192" rot="R90"/>
 <element name="R12" library="RCL" package="0603" value="330R" x="27.94" y="14.732" rot="R270"/>
@@
 <vertex x="0.118" y="0"/>
 </polygon>
-<contactref element="R10" pad="1"/>
-<contactref element="SV1" pad="5"/>
 <contactref element="R17" pad="1"/>
-<contactref element="R11" pad="1"/>
 <contactref element="R12" pad="1"/>
 <contactref element="R13" pad="1"/>
@@
 <signal name="N$23">
 </signal>
-<signal name="N$13">
-<contactref element="LED1" pad="1"/>
-<contactref element="SV1" pad="1"/>
-<wire x1="35.941" y1="9.906" x2="37.465" y2="9.906" width="0.254" layer="1"/>
-<wire x1="37.465" y1="9.906" x2="37.964" y2="9.906" width="0.6096" layer="1"/>
-<wire x1="37.964" y1="9.906" x2="39.234" y2="8.636" width="0.6096" layer="1"/>
-<wire x1="35.941" y1="9.906" x2="31.496" y2="9.906" width="0.6096" layer="1"/>
-<wire x1="31.496" y1="9.906" x2="30.48" y2="10.922" width="0.6096" layer="1"/>
-<wire x1="30.48" y1="11.4946" x2="30.48" y2="10.922" width="0.6096" layer="1"/>
-</signal>
-<signal name="N$14">
-<contactref element="R10" pad="2"/>
-<contactref element="LED1" pad="2"/>
-<wire x1="30.48" y1="12.8894" x2="30.48" y2="14.0346" width="0.6096" layer="1"/>
-</signal>
-<signal name="N$15">
-<contactref element="R11" pad="2"/>
-<contactref element="LED2" pad="2"/>
-<wire x1="29.21" y1="12.8894" x2="29.21" y2="14.0346" width="0.6096" layer="1"/>
-</signal>
 <signal name="N$16">
 <contactref element="R12" pad="2"/>
@@
 <contactref element="LED8" pad="2"/>
 <wire x1="21.59" y1="12.8894" x2="21.59" y2="14.0346" width="0.6096" layer="1"/>
-</signal>
-<signal name="N$29">
-<contactref element="LED2" pad="1"/>
-<contactref element="SV1" pad="2"/>
-<wire x1="36.694" y1="8.636" x2="31.369" y2="8.636" width="0.6096" layer="1"/>
-<wire x1="31.369" y1="8.636" x2="29.21" y2="10.795" width="0.6096" layer="1"/>
-<wire x1="29.21" y1="10.795" x2="29.21" y2="11.4946" width="0.6096" layer="1"/>
-</signal>
-<signal name="N$30">
-<contactref element="LED3" pad="1"/>
-<contactref element="SV1" pad="3"/>
-<wire x1="31.496" y1="7.112" x2="39.878" y2="7.112" width="0.6096" layer="1"/>
-<wire x1="39.878" y1="7.112" x2="40.767" y2="8.001" width="0.6096" layer="1"/>
-<wire x1="40.767" y1="8.001" x2="40.767" y2="9.643" width="0.6096" layer="1"/>
-<wire x1="40.767" y1="9.643" x2="39.234" y2="11.176" width="0.6096" layer="1"/>
-<wire x1="31.496" y1="7.112" x2="27.94" y2="10.668" width="0.6096" layer="1"/>
-<wire x1="27.94" y1="10.668" x2="27.94" y2="11.4946" width="0.6096" layer="1"/>
-</signal>
-<signal name="N$31">
-<contactref element="LED4" pad="1"/>
-<contactref element="SV1" pad="4"/>
-<wire x1="31.115" y1="6.096" x2="40.259" y2="6.096" width="0.6096" layer="1"/>
-<wire x1="40.259" y1="6.096" x2="41.783" y2="7.62" width="0.6096" layer="1"/>
-<wire x1="41.783" y1="7.62" x2="41.783" y2="10.795" width="0.6096" layer="1"/>
-<wire x1="41.783" y1="10.795" x2="40.132" y2="12.446" width="0.6096" layer="1"/>
-<wire x1="40.132" y1="12.446" x2="40.005" y2="12.446" width="0.6096" layer="1"/>
-<wire x1="40.005" y1="12.446" x2="38.481" y2="12.446" width="0.254" layer="1"/>
-<wire x1="38.481" y1="12.446" x2="37.964" y2="12.446" width="0.6096" layer="1"/>
-<wire x1="37.964" y1="12.446" x2="36.694" y2="11.176" width="0.6096" layer="1"/>
-<wire x1="31.115" y1="6.096" x2="26.67" y2="10.541" width="0.6096" layer="1"/>
-<wire x1="26.67" y1="10.541" x2="26.67" y2="11.4946" width="0.6096" layer="1"/>
 </signal>
 <signal name="N$32">
@@
 <contactref element="OUT" pad="P$19"/>
 <wire x1="26.67" y1="5.08" x2="26.67" y2="19.431" width="0.6096" layer="16"/>
+<contactref element="LED4" pad="1"/>
+<wire x1="26.67" y1="5.08" x2="26.67" y2="11.4946" width="0.6096" layer="1"/>
 </signal>
 <signal name="N$2">
@@
 <wire x1="28.194" y1="4.064" x2="28.194" y2="20.447" width="0.6096" layer="16"/>
 <wire x1="28.194" y1="20.447" x2="26.67" y2="21.971" width="0.6096" layer="16"/>
+<contactref element="LED3" pad="1"/>
+<wire x1="27.94" y1="11.4946" x2="27.94" y2="6.223" width="0.6096" layer="1"/>
+<wire x1="27.94" y1="6.223" x2="28.194" y2="5.969" width="0.6096" layer="1"/>
+<wire x1="28.194" y1="5.969" x2="28.194" y2="4.064" width="0.6096" layer="1"/>
+<wire x1="28.194" y1="4.064" x2="26.67" y2="2.54" width="0.6096" layer="1"/>
 </signal>
 <signal name="N$3">
