File: Other/EXT_LED.sch (EAGLE design)
At the start: 39 parts

Commit message: Minor Changes
Parts:
- removed LED1, LED2: (no value), Optic:LED0603
- removed R10, R11: 330R, RCL:R0603
- removed SV1: (no value), Conn:ML6ES
Connections:
- removed net N$13: LED1.A, SV1-1.S
- removed net N$14: LED1.C, R10.2
- removed net N$15: LED2.C, R11.2
- removed net N$29: LED2.A, SV1-2.S
- removed net N$30: LED3.A, SV1-3.S
- removed net N$31: LED4.A, SV1-4.S
- net GND: no longer R10.1, R11.1, SV1-5.S
- net N$1: now also LED4.A
- net N$2: now also LED3.A
Other:
- moved on the sheet: IN-19, IN-20, OUT-19, OUT-20
